File: PCB/PCB_v1.1.brd (EAGLE design)
At the start: 31.8 x 20 mm, 15 parts, among them Q1 NPN, Q2 NPN, SW1 MLL1200S

Commit message: Fix schematic
Parts:
- removed D2, D3: LED_BLUE, LED:LEDC1608X55N_FLAT-B
- removed R4: 12K, Resistor:RESC1608X60
- removed R5, R6: 1.5K, Resistor:RESC1608X60
- removed R7: 4.7K, Resistor:RESC1608X60
- D1: value LED_BLUE -> LED_GREEN
- R1, R2: value 470R -> 12K
- R3: value 12K -> 4.7K
- moved R1 3.81 mm to (-7.62, 16.5)
- moved R2 3.81 mm to (-7.62, 14.0)
- moved R3 3.81 mm to (-7.62, 11.4)
- moved D1 1.27 mm to (-7.62, 16.5)
- moved Q1 1.27 mm to (0.00, 14.0)
- moved Q2 1.27 mm to (6.35, 14.0)
Connections:
- removed net ESP_RX: ESPF.3, R1.2
- removed net ESP_TX: ESPF.2, R2.2
- removed net N$2: D1.A, R5.1
- removed net N$4: D2.A, R6.1
- removed net N$6: D3.A, R7.1
- new net N$1: D1.C, R3.1
- net DTR: now also R1.1; no longer R3.1
- net ESP_3.3V: now also D1.A; no longer D3.C
- net FLIPPER_RX: now also ESPF.2; no longer D1.C, R2.1
- net FLIPPER_TX: now also ESPF.3; no longer D2.C, R1.1
- net GND: now also R3.2; no longer R5.2, R6.2, R7.2
- net N$3: now also R1.2; no longer R3.2
- net N$5: now also R2.2; no longer R4.2
- net RTS: now also R2.1; no longer R4.1
Routing:
- net FLIPPER_RX: track 37.4 -> 5.86 mm, vias 1 -> 0
- net N$3: track 37.5 -> 10.2 mm
- net FLIPPER_TX: track 30.4 -> 7.94 mm, vias 1 -> 0
- net ESP_RX: track 19.2 -> 0.00 mm
- net RTS: track 36.5 -> 19.6 mm, vias 0 -> 1
- net ESP_TX: track 15.3 -> 0.00 mm
- net N$5: track 15.4 -> 29.8 mm
- net GND: track 49.0 -> 39.9 mm, vias 1 -> 0
- net N$1: track 0.00 -> 7.74 mm, vias 0 -> 1
- net N$2: track 3.49 -> 0.00 mm, vias 1 -> 0
- net DTR: track 39.4 -> 35.9 mm
- net N$4: track 2.15 -> 0.00 mm, vias 1 -> 0
- net N$6: track 2.05 -> 0.00 mm, vias 1 -> 0
- net 3.3V: track 7.99 -> 9.04 mm
- net GPIO0: track 6.18 -> 5.40 mm
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Other:
- board text added: "3.3V Status"
- board text added: "Flipper Zero Flasher Board v1.1 by Oleksii Kutuzov"
- board text added: "GND RX TX 3.3V EN IO0"
- board text added: "OFF ON"
- board text removed: "3.3V"
- board text removed: "Flipper Zero Flasher Board v1.0 by Oleksii Kutuzov"
- board text removed: "GND TX RX 3.3V EN IO0"
- board text removed: "OFF ON 3.3V"
- board text removed: "RX"
- board text removed: "TX"
