File: PCB/Schematic_v1.1.sch (EAGLE design)
At the start: 15 parts, among them Q1 NPN, Q2 NPN, SW1 MLL1200S

Commit message: Fix schematic
Parts:
- removed D2, D3: LED_BLUE, LED:CHIP-FLAT-B_0603-0.55MM
- removed R4: 12K, Resistor:R_CHIP-0603(1608-METRIC)
- removed R5, R6: 1.5K, Resistor:R_CHIP-0603(1608-METRIC)
- removed R7: 4.7K, Resistor:R_CHIP-0603(1608-METRIC)
- D1: value LED_BLUE -> LED_GREEN
- R1, R2: value 470R -> 12K
- R3: value 12K -> 4.7K
Connections:
- removed net ESP_RX: ESPF.ESP_RX, R1.2
- removed net ESP_TX: ESPF.ESP_TX, R2.2
- removed net N$2: D1.A, R5.1
- removed net N$4: D2.A, R6.1
- removed net N$6: D3.A, R7.1
- new net N$1: D1.C, R3.1
- net DTR: now also R1.1; no longer R3.1
- net ESP_3.3V: now also D1.A; no longer D3.C
- net FLIPPER_RX: now also ESPF.ESP_TX; no longer D1.C, R2.1
- net FLIPPER_TX: now also ESPF.ESP_RX; no longer D2.C, R1.1
- net GND: now also R3.2; no longer R5.2, R6.2, R7.2
- net N$3: now also R1.2; no longer R3.2
- net N$5: now also R2.2; no longer R4.2
- net RTS: now also R2.1; no longer R4.1
Other:
- moved on the sheet: D1, R1, R2, R3
